File: kicad/interposer.kicad_sch (KiCad schematic)
At the start: 9 parts, among them J1 Conn_Stove, U1 XIAO-nRF52840, U2 Adafruit DS3502, U3 TS5A3159DBV

Commit message: Update KiCad to two layers
Parts:
- B1: renamed from LS1; value Speaker -> Buzzer
Connections:
- net BYPASS: now also U1.11 (PA6_A10_D10_MOSI); no longer U1.2 (PA4_A1_D1)
- net GND: now also J1.3 (Pin_3); no longer J1.2 (Pin_2)
- net INPUT: now also U1.5 (PA8_A4_D4_SDA); no longer U1.1 (PA02_A0_D0)
- net KNOB: now also J1.4 (Pin_4); no longer J1.3 (Pin_3)
- net RETURN: now also J1.2 (Pin_2); no longer J1.4 (Pin_4)
- net at U1.10 (PA5_A9_D9_MISO): no longer B1.2
- net at B1.1: now also U1.1 (PA02_A0_D0); no longer U1.11 (PA6_A10_D10_MOSI)
- new net: B1.2, U1.2 (PA4_A1_D1)
Other:
- moved on the sheet: B1, J1, U1, U2

Commit message: Update KiCad
Parts:
- removed B1: Buzzer, Buzzer_Beeper:Buzzer_TDK_PS1240P02BT_D12.2mm_H6.5mm, symbol library:Speaker
- removed C1: 0.1µF, Capacitor_THT:C_Disc_D5.0mm_W2.5mm_P5.00mm, symbol library:C
- removed J1: Conn_Stove, Connector_PinHeader_2.54mm:PinHeader_1x04_P2.54mm_Vertical, symbol library:Conn_01x04
- removed R1, R3: 10kΩ, Resistor_THT:R_Axial_DIN0207_L6.3mm_D2.5mm_P10.16mm_Horizontal, symbol library:R
- removed R2: 18kΩ, Resistor_THT:R_Axial_DIN0207_L6.3mm_D2.5mm_P10.16mm_Horizontal, symbol library:R
- removed U1: XIAO-nRF52840, Package_DIP:DIP-14_W7.62mm, symbol library:XIAO-nRF52840-DIP
- removed U2: Adafruit DS3502, Package_DIP:DIP-12_W7.62mm, symbol library:DS3502
- removed U3: TS5A3159DBV, Package_DIP:DIP-6_W7.62mm, symbol library:TS5A3159DBV
- added B1: Buzzer, interposer:Buzzer_TDK_PS1240P02BT_D12.2mm_H6.5mm, symbol Device:Speaker
- added C1, C2: 100nF, Capacitor_SMD:C_0805_2012Metric_Pad1.18x1.45mm_HandSolder, symbol Device:C
- added C3, C4: 1µF, Capacitor_SMD:C_0805_2012Metric_Pad1.18x1.45mm_HandSolder, symbol Device:C
- added J1: Dial, Connector_JST:JST_XH_B3B-XH-A_1x03_P2.50mm_Vertical, symbol Connector_Generic:Conn_01x03
- added J2: Stove, Connector_JST:JST_XH_B3B-XH-A_1x03_P2.50mm_Vertical, symbol Connector_Generic:Conn_01x03
- added J3: Stove, Connector_JST:JST_XH_S3B-XH-A_1x03_P2.50mm_Horizontal, symbol Connector_Generic:Conn_01x03
- added Q1: 2N7002, Package_TO_SOT_SMD:SOT-23, symbol Transistor_FET:2N7002
- added R1, R3: 27kΩ, Resistor_SMD:R_0805_2012Metric_Pad1.20x1.40mm_HandSolder, symbol Device:R
- added R2, R4: 51kΩ, Resistor_SMD:R_0805_2012Metric_Pad1.20x1.40mm_HandSolder, symbol Device:R
- added R5: 33kΩ, Resistor_SMD:R_0805_2012Metric_Pad1.20x1.40mm_HandSolder, symbol Device:R
- added R6: 100kΩ, Resistor_SMD:R_0805_2012Metric_Pad1.20x1.40mm_HandSolder, symbol Device:R
- added R7: 100Ω, Resistor_SMD:R_0805_2012Metric_Pad1.20x1.40mm_HandSolder, symbol Device:R
- added R8: 1MΩ, Resistor_SMD:R_0805_2012Metric_Pad1.20x1.40mm_HandSolder, symbol Device:R
- added U1: XIAO-nRF52840-DIP, interposer:XIAO-nRF52840-DIP, symbol Seeed_Studio_XIAO_Series:XIAO-nRF52840-DIP
- added U2: MCP6042-E_SN, Package_SO:SOIC-8_3.9x4.9mm_P1.27mm, symbol interposer:MCP6042-E_SN
- added U3: TXU0101DBVR, Package_TO_SOT_SMD:SOT-23-6_Handsoldering, symbol interposer:TXU0101DBVR
- added U4: TMUX1119DBVR, Package_TO_SOT_SMD:SOT-23-6_Handsoldering, symbol interposer:TMUX1119DBVR
Connections:
- net +3V3: now also U1.12 (3V3), U3.1 (VCCA), U3.5 (OE)
- net +5V: now also C4.1, J1.1 (Pin_1), J2.3 (Pin_3), R1.1, U2.8 (VDD), U3.6 (VCCB), U4.2 (V+)
- net GND: now also C1.2, C2.2, C3.2, C4.2, J1.3 (Pin_3), J2.1 (Pin_1), Q1.2 (S), R2.2, R4.2, R6.2, U1.13 (GND), U2.4 (VSS), U3.2 (GND), U4.3 (GND)
- new net: Q1.3 (D), R8.2
- new net: B1.1, R7.1
- new net +BUZZ: R7.2, U1.2 (P0.03_A1_D1)
- new net -BUZZ: B1.2, U1.3 (P0.28_A2_D2)
- new net DIAL: J1.2 (Pin_2), R8.1, U2.3 (VINA+), U4.4 (NC)
- new net IN: R3.1, U2.1 (VOUTA), U2.2 (VINA-)
- new net OUT: U2.6 (VINB-), U2.7 (VOUTB), U4.6 (NO)
- new net PWM_3V3: U1.1 (P0.02_A0_D0), U3.3 (A)
- new net PWM_5V: R5.1, U3.4 (BY)
- new net RC: C3.1, R5.2, U2.5 (VINB+)
- new net READ: C2.1, R3.2, R4.1, U1.4 (P0.29_A3_D3)
- new net REF: C1.1, R1.2, R2.1, U1.5 (P0.04_A4_D4_SDA)
- new net SEL: Q1.1 (G), R6.1, U1.11 (P1.15_D10_MOSI), U4.1 (SEL)
- new net STOVE: J2.2 (Pin_2), U4.5 (COM)
- no-connect marks 0 -> 9
