File: kicad/interposer.kicad_sch (KiCad schematic)
At the start: 21 parts, among them J1 Dial, J2 Stove, J3 Stove, Q1 2N7002, U1 XIAO-nRF52840-DIP, U2 MCP6042-E_SN, U3 TXU0101DBVR, U4 TMUX1119DBVR

Commit message: Update KiCad
Parts:
- removed J2: Stove, Connector_JST:JST_XH_B3B-XH-A_1x03_P2.50mm_Vertical, symbol Connector_Generic:Conn_01x03
- removed J3: Stove, Connector_JST:JST_XH_S3B-XH-A_1x03_P2.50mm_Horizontal, symbol Connector_Generic:Conn_01x03
- removed Q1: 2N7002, Package_TO_SOT_SMD:SOT-23, symbol Transistor_FET:2N7002
- removed R1: 27kΩ, Resistor_SMD:R_0805_2012Metric_Pad1.20x1.40mm_HandSolder, symbol Device:R
- removed R5: 33kΩ, Resistor_SMD:R_0805_2012Metric_Pad1.20x1.40mm_HandSolder, symbol Device:R
- removed R6: 100kΩ, Resistor_SMD:R_0805_2012Metric_Pad1.20x1.40mm_HandSolder, symbol Device:R
- removed R8: 1MΩ, Resistor_SMD:R_0805_2012Metric_Pad1.20x1.40mm_HandSolder, symbol Device:R
- removed U2: MCP6042-E_SN, Package_SO:SOIC-8_3.9x4.9mm_P1.27mm, symbol interposer:MCP6042-E_SN
- removed U3: TXU0101DBVR, Package_TO_SOT_SMD:SOT-23-6_Handsoldering, symbol interposer:TXU0101DBVR
- removed U4: TMUX1119DBVR, Package_TO_SOT_SMD:SOT-23-6_Handsoldering, symbol interposer:TMUX1119DBVR
- added IC1: PIC16F17114-I_SN, Package_SO:SOIC-8_3.9x4.9mm_P1.27mm, symbol interposer:PIC16F17114-I_SN
- added IC2: ISO7021DR, Package_SO:SOIC-8_3.9x4.9mm_P1.27mm, symbol interposer:ISO7021DR
- added J1: PADS_STOVE_SIG, interposer:RAST 2.5 Pads, symbol Connector_Generic:Conn_01x03
- added J3: USB_PIC, interposer:SAMESKY_UJ20-C-H-G-SMT-P16-TR, symbol interposer:UJ20-C-H-G-SMT-P16-TR
- added J4: USB_XIAO, interposer:SAMESKY_UJ20-C-H-G-SMT-P16-TR, symbol interposer:UJ20-C-H-G-SMT-P16-TR
- B1: footprint interposer:Buzzer_TDK_PS1240P02BT_D12.2mm_H6.5mm -> Buzzer_Beeper:Buzzer_Murata_PKLCS1212E
- C1: value 100nF -> 10µF
- C3: value 1µF -> 10nF
- C4: value 1µF -> 100nF
- J2: renamed from J1; value Dial -> JST_DIAL; footprint Connector_JST:JST_XH_B3B-XH-A_1x03_P2.50mm_Vertical -> Connector_JST:JST_XH_S3B-XH-A_1x03_P2.50mm_Horizontal
- R1: renamed from R7; value 100Ω -> 220Ω
- R2: value 51kΩ -> 10kΩ
- R3: value 27kΩ -> 220Ω
- R4: value 51kΩ -> 270kΩ
Connections:
- net RC is gone; now on net DIAL_REF: C3.1
- net +3V3: now also J4.A4_B9 (VBUS), J4.B4_A9 (VBUS)
- net +5V: now also C1.1, C2.1, R2.2, IC1.1 (VDD), IC2.1 (VCC1), J1.1 (Pin_1); no longer C4.1, J2.1 (Pin_1)
- net +BUZZ: now also U1.3 (P0.28_A2_D2); no longer U1.2 (P0.03_A1_D1)
- net -BUZZ: now also U1.4 (P0.29_A3_D3); no longer U1.3 (P0.28_A2_D2)
- net DIAL renamed DIAL_SIG
- net DIAL_SIG: now also R4.1, IC1.3 (RA4)
- net GND renamed GND_PIC
- net GND_PIC: now also J2.1 (Pin_1), IC1.8 (VSS), IC2.4 (GND1), J1.3 (Pin_3); no longer C4.2, J2.3 (Pin_3), R2.2, U1.13 (GND)
- net IN renamed DIAL_REF
- net DIAL_REF: now also J2.3 (Pin_3)
- net PWM_3V3 renamed RX_XIAO
- net RX_XIAO: now also J4.A6 (DP1), J4.B6 (DP2)
- removed net READ: C2.1, R3.2, R4.1, U1.4 (P0.29_A3_D3)
- removed net REF: C1.1, R2.1, U1.5 (P0.04_A4_D4_SDA)
- net SEL renamed PROG_XIAO
- net PROG_XIAO: now also J4.A8 (SBU1), J4.B8 (SBU2)
- new net: J3.SH1 (SHIELD), J3.SH2 (SHIELD), J3.SH3 (SHIELD), J3.SH4 (SHIELD)
- new net DIAL_EXC: IC1.2 (RA5), R3.2
- new net GND_ISO: C4.2, IC2.5 (GND2), J3.A12_B1 (GND), J3.A1_B12 (GND)
- new net GND_XIAO: J4.A12_B1 (GND), J4.A1_B12 (GND), J4.SH1 (SHIELD), J4.SH2 (SHIELD), J4.SH3 (SHIELD), J4.SH4 (SHIELD), U1.13 (GND)
- new net PROG_PIC: IC1.4 (~{MCLR}/VPP/RA3), J3.A8 (SBU1), J3.B8 (SBU2), R2.1
- new net RX_ISO: IC2.6 (OUTB), J3.A6 (DP1), J3.B6 (DP2)
- new net RX_PIC: IC1.7 (RA0/ICSPDAT), IC2.2 (OUTA)
- new net STOVE_SIG: IC1.5 (RA2), J1.2 (Pin_2)
- new net TX_ISO: IC2.7 (INA), J3.A7 (DN1), J3.B7 (DN2)
- new net TX_PIC: IC1.6 (RA1/ICSPCLK), IC2.3 (INB)
- new net TX_XIAO: J4.A7 (DN1), J4.B7 (DN2), U1.2 (P0.03_A1_D1)
- new net VBUS_ISO: C4.1, IC2.8 (VCC2), J3.A4_B9 (VBUS), J3.B4_A9 (VBUS)
- no-connect marks 9 -> 12
Other:
- moved on the sheet: B1, J2, R1, U1
